Commit message: add STS3215 controller, add a Intel RealSense D405 camera

File: src/lerobot_description/urdf/so101.urdf.xacro (robot description, xacro)
@@ -1,4 +1,5 @@
 <?xml version="1.0"?>
 <robot name="so101" xmlns:xacro="http://www.ros.org/wiki/xacro">
+    <xacro:arg name="use_sim" default="false" />
     <xacro:include filename="$(find lerobot_description)/urdf/so101_base.xacro" />
     <xacro:include filename="$(find lerobot_description)/urdf/so101_gazebo.xacro" />

File: src/lerobot_description/urdf/so101_base.xacro (robot description, xacro)
@@ -6,4 +6,5 @@
 -->
 <robot xmlns:xacro="http://www.ros.org/wiki/xacro">
+	<xacro:include filename="$(find realsense2_description)/urdf/_d405.urdf.xacro" />
 	<!-- Links -->
 	<link name="world" />
@@ -341,4 +342,5 @@
 	<!-- Joint from gripper to jaw -->
 	<joint name="6" type="revolute">
+		<param name="motor_id">6</param>
 		<origin xyz="0.0202 0.0188 -0.0234" rpy="1.5708 -5.14108e-17 -1.38655e-14" />
 		<parent link="gripper" />
@@ -359,4 +361,5 @@
 	<!-- Joint from wrist to gripper -->
 	<joint name="5" type="revolute">
+		<param name="motor_id">5</param>
 		<origin xyz="0 -0.0611 0.0181" rpy="1.5708 -9.38083e-08 3.14159" />
 		<parent link="wrist" />
@@ -377,4 +380,5 @@
 	<!-- Joint from lower_arm to wrist -->
 	<joint name="4" type="revolute">
+		<param name="motor_id">4</param>
 		<origin xyz="-0.1349 0.0052 1.65232e-16" rpy="3.2474e-15 2.86219e-15 -1.5708" />
 		<parent link="lower_arm" />
@@ -395,9 +399,10 @@
 	<!-- Joint from upper_arm to lower_arm -->
 	<joint name="3" type="revolute">
+		<param name="motor_id">3</param>
 		<origin xyz="-0.11257 -0.028 2.46331e-16" rpy="-1.22818e-15 5.75928e-16 1.5708" />
 		<parent link="upper_arm" />
 		<child link="lower_arm" />
 		<axis xyz="0 0 1" />
-		<limit effort="10" velocity="10" lower="-1.74533" upper="1.5708" />
+		<limit effort="10" velocity="10" lower="-1.74" upper="1.8" />
 	</joint>
 	<transmission name="3_trans">
@@ -413,9 +418,10 @@
 	<!-- Joint from shoulder to upper_arm -->
 	<joint name="2" type="revolute">
+		<param name="motor_id">2</param>
 		<origin xyz="-0.0303992 -0.0182778 -0.0542" rpy="-1.5708 -1.5708 0" />
 		<parent link="shoulder" />
 		<child link="upper_arm" />
 		<axis xyz="0 0 1" />
-		<limit effort="10" velocity="10" lower="-1.74533" upper="1.74533" />
+		<limit effort="10" velocity="10" lower="-2.0" upper="2.0" />
 	</joint>
 	<transmission name="2_trans">
@@ -431,4 +437,5 @@
 	<!-- Joint from base to shoulder -->
 	<joint name="1" type="revolute">
+		<param name="motor_id">1</param>
 		<origin xyz="0.0207909 -0.0230745 0.0948817" rpy="-3.14159 6.03684e-16 1.5708" />
 		<parent link="base" />
@@ -447,3 +454,12 @@
 		</actuator>
 	</transmission>
+	<link name="camera_mount_point" />
+    <joint name="gripper_to_camera_mount" type="fixed">
+        <parent link="gripper" />
+        <child link="camera_mount_point" />
+        <origin xyz="0.0 0.0 0.0" rpy="0.0 0.0 0.0" />
+    </joint>
+    <xacro:sensor_d405 parent="camera_mount_point" name="camera" use_nominal_extrinsics="true">
+        <origin xyz="0 0 0" rpy="0 0 0"/>
+    </xacro:sensor_d405>
 </robot>

File: src/lerobot_description/urdf/so101_gazebo.xacro (robot description, xacro)
@@ -1,9 +1,11 @@
 <?xml version="1.0"?>
 <robot xmlns:xacro="http://www.ros.org/wiki/xacro">
-    <!-- ROS 2 Control -->
-    <gazebo>
-        <plugin filename="gz_ros2_control-system" name="gz_ros2_control::GazeboSimROS2ControlPlugin">
-            <parameters>$(find lerobot_controller)/config/so101_controllers.yaml</parameters>
-        </plugin>
-    </gazebo>
+    <xacro:arg name="use_sim" default="false" />
+    <xacro:if value="$(arg use_sim)">
+        <gazebo>
+            <plugin filename="gz_ros2_control-system" name="gz_ros2_control::GazeboSimROS2ControlPlugin">
+                <parameters>$(find lerobot_controller)/config/so101_controllers.yaml</parameters>
+            </plugin>
+        </gazebo>
+    </xacro:if>
 </robot>

File: src/lerobot_description/urdf/so101_ros2_control.xacro (robot description, xacro)
@@ -1,10 +1,20 @@
 <?xml version="1.0"?>
 <robot xmlns:xacro="http://www.ros.org/wiki/xacro">
+    <xacro:arg name="use_sim" default="false" />
     <ros2_control name="RobotSystem" type="system">
-        <!-- ros2_control Gazebo -->
-        <hardware>
-            <plugin>gz_ros2_control/GazeboSimSystem</plugin>
-        </hardware>
+        <xacro:if value="$(arg use_sim)">
+            <hardware>
+                <plugin>gz_ros2_control/GazeboSimSystem</plugin>
+            </hardware>
+        </xacro:if>
+        <xacro:unless value="$(arg use_sim)">
+            <hardware>
+                <plugin>so101_hardware/STS3215HardwareInterface</plugin>
+                <param name="usb_port">/dev/ttyUSB0</param>
+                <param name="baud_rate">1000000</param>
+            </hardware>
+        </xacro:unless>
         <joint name="1">
+            <param name="motor_id">1</param>
             <command_interface name="position">
                 <param name="min">-1.91986</param>
@@ -12,20 +22,26 @@
             </command_interface>
             <state_interface name="position" />
+            <state_interface name="velocity" />
         </joint>
         <joint name="2">
+            <param name="motor_id">2</param>
             <command_interface name="position">
-                <param name="min">-1.74533</param>
-                <param name="max">1.74533</param>
+                <param name="min">-2.0</param>
+                <param name="max">2.0</param>
             </command_interface>
             <state_interface name="position" />
+            <state_interface name="velocity" />
         </joint>
         <joint name="3">
+            <param name="motor_id">3</param>
             <command_interface name="position">
-                <param name="min">-1.74533</param>
-                <param name="max">1.5708</param>
+                <param name="min">-1.74</param>
+                <param name="max">1.8</param>
             </command_interface>
             <state_interface name="position" />
+            <state_interface name="velocity" />
         </joint>
         <joint name="4">
+            <param name="motor_id">4</param>
             <command_interface name="position">
                 <param name="min">-1.65806</param>
@@ -33,6 +49,8 @@
             </command_interface>
             <state_interface name="position" />
+            <state_interface name="velocity" />
         </joint>
         <joint name="5">
+            <param name="motor_id">5</param>
             <command_interface name="position">
                 <param name="min">-2.79253</param>
@@ -40,6 +58,8 @@
             </command_interface>
             <state_interface name="position" />
+            <state_interface name="velocity" />
         </joint>
         <joint name="6">
+            <param name="motor_id">6</param>
             <command_interface name="position">
                 <param name="min">-0.174533</param>
@@ -47,4 +67,5 @@
             </command_interface>
             <state_interface name="position" />
+            <state_interface name="velocity" />
         </joint>
     </ros2_control>
