Commit message: Initial commit

File: src/lerobot_description/urdf/so101_base.xacro (robot description, xacro)
@@ -366,5 +366,5 @@
 		<child link="gripper" />
 		<axis xyz="0 0 1" />
-		<limit effort="10" velocity="10" lower="-2.79253" upper="2.79253" />
+		<limit effort="10" velocity="10" lower="-3.0" upper="3.0" />
 	</joint>
 	<transmission name="5_trans">
@@ -385,5 +385,5 @@
 		<child link="wrist" />
 		<axis xyz="0 0 1" />
-		<limit effort="10" velocity="10" lower="-1.65806" upper="1.65806" />
+		<limit effort="10" velocity="10" lower="-2.0" upper="2.0" />
 	</joint>
 	<transmission name="4_trans">
@@ -442,5 +442,5 @@
 		<child link="shoulder" />
 		<axis xyz="0 0 1" />
-		<limit effort="10" velocity="10" lower="-1.91986" upper="1.91986" />
+		<limit effort="10" velocity="10" lower="-2.0" upper="2.0" />
 	</joint>
 	<transmission name="1_trans">
